Commit message: 增加运动学解算程序

File: 3.Software/ROS package/HotDog/urdf/HotDog.urdf (robot description, URDF)
Before this commit: robot HotDog, 25 links, 24 joints
Joints:
- removed joint LF_R_JOIN
- added joint LF_R_JOINT: type revolute, parent LF_SHANK_LINK, child LF_R_LINK, origin xyz=0.122 0 0 rpy=1.5708 0 0, axis 0 0 -1, limit lower=-1.5708 upper=1.5708 effort=0 velocity=0
